File: catpaw.kicad_sch (KiCad schematic)
At the start: 26 parts, among them J1 m12,Acode,5pin,femalesocket, J3 Conn_01x01_Socket, J4 Conn_01x01_Socket, SW1 SW_DPST, U1 INA826, U2 ${SIM.PARAMS}

Commit message: scheme rework
Parts:
- added J4: m8, 4Pin Supply Connector, symbol Connector:Conn_01x04_Socket
- added J5: m8, 4Pin Supply Connector Beckhoff, symbol Connector:Conn_01x04_Socket
- added J6: m12,Acode,5pin,femalesocket Beckhoff INPUT, symbol Connector:Conn_01x05_Socket
- added R50: 3M, symbol Device:R
- added R51: 27k-30k, symbol Device:R
- J1: renamed from J4; value Conn_01x01_Socket -> Conn_01x01_Socket_red
- J2: renamed from J3; value Conn_01x01_Socket -> Conn_01x01_Socket_black
- J3: renamed from J1; value m12,Acode,5pin,femalesocket -> m12,Acode,5pin,femalesocket (to Input)
- R1, R2, R3, R5, R6, R7: value 680k -> 1M
- R4: value 39k -> 30k
Connections:
- net GND: now also J6.4 (Pin_4); no longer D3.1 (K), J3.3 (Pin_3), J3.5 (Pin_5), PS1.4 (-Vout), R13.2, R15.1, U1.5 (Vs-), U2.4 (V-)
- net pwrout+ renamed Up Peripheral V
- net Up Peripheral V: now also J3.1 (Pin_1), J4.2 (Pin_2), J5.2 (Pin_2), J6.1 (Pin_1); no longer C2.2, J3.2 (Pin_2)
- net sigout+ renamed In+ Analog Input
- net In+ Analog Input: now also J3.2 (Pin_2), J6.2 (Pin_2); no longer J3.1 (Pin_1)
- new net: R50.2, R51.1
- new net: R50.1, R51.2
- new net GNDp: C2.2, D3.1 (K), J3.3 (Pin_3), J4.4 (Pin_4), J5.4 (Pin_4), J6.3 (Pin_3), PS1.4 (-Vout), R13.2, R15.1, U1.5 (Vs-), U2.4 (V-)
- new net GNDs: J5.3 (Pin_3)
- new net Shield: J6.5 (Pin_5)
- new net Us Control V: J5.1 (Pin_1)
- new net cable shield: J3.5 (Pin_5)
- no-connect marks 0 -> 2
Other:
- added sheet scribble (scribble.kicad_sch)
- note added: "7/14/26 480*62000 / (3000000+62000) = 9.72V note gain will equal 2 9.72v * 2 = 19.44 so: R4 = 30k, Vout = 4.75v with gain of 2 = 9.5V"
- note added: "7/14/26 beckhoff analog i/o have common analog gnd which is isolated from all other grounds in box EP4274-0002, 3.2 page 12"
- note added: "BECKHOFF REFERENCES"
- note added: "R8/11 derived from ina826 datasheet"
- note added: "Up is for Ext Sensor on analog input 1,2 we need Us to get to the beckhoff for processor logic field bus & analog i/0"
- note added: "Vout= G X (Vin+ - Vin-) G = 1 + 49.4k / Rg) G = 2"
- note added: "bananajack pair double check placement"
- note added: "divider setup to make 480vac =<5V"
- note added: "double check Rg formula, appears gain cannot be equal to or lower than 1 Gain will equal 2 rework divider network to lower input voltage, use 1M 1206 resistors calculate new R4 value"
- note added: "pwrout+/2 divider at ref datasheet:8.3.7"
- note added: "thruhole LED panelmount"
- note added: "tie pwrout- to devicecommon gnd? check m12 acode pinout -nope-"
- note added: "update: 06/04/26"
- note added: "with the ref divider sigout- and pwrout- are at two different potentials sigout- is directly between pwr +/-, it is gnd double check the beckoff manual"
- note removed: "bananajack pair"
- note removed: "consider pwrout+/2 divider at ref datasheet:8.3.7"
- note removed: "divider setup to make 480vac =<10V"
- note removed: "double check Rg formula, appears gain cannot be equal to or lower than 1 consider reworking divider network to lower input voltage"
- note removed: "thruhole LED"
- note removed: "tie pwrout- to devicecommon gnd? check m12 acode pinout"
- moved on the sheet: C1, C2, D3, F1, J1, J2, J3, PS1, R1, R10, R11, R12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

Commit message: added M8 connector to RAK psu output
Parts:
- added D1, D2, D3, D4: 1N5819, Diode_THT:D_DO-41_SOD81_P10.16mm_Horizontal, symbol Diode:1N5819
- added J3: m12,Acode,5pin,femalesocket (to beckhoff input), symbol Connector:Conn_01x05_Socket
- J4: value m8, 4Pin Supply Connector -> m8, 4Pin Supply Connector FEMALE
- J7: renamed from J3; value m12,Acode,5pin,femalesocket (to Input) -> m12,Acode,5pin,femalesocket CATPAW; now left out of the parts list
- R12: value 2.2k -> 4.7k
- renumbered D3 to D5
Connections:
- net GND: now also J3.4 (Pin_4)
- net GNDp: no longer C2.2, D5.1 (K), J4.4 (Pin_4), PS1.4 (-Vout), R13.2, R15.1, U1.5 (Vs-), U2.4 (V-)
- net In+ Analog Input: now also J3.2 (Pin_2)
- net Up Peripheral V: no longer C1.2, J4.2 (Pin_2), PS1.5 (+Vout), R12.2, R14.2, U1.8 (Vs+), U2.3 (V+)
- net cable shield: now also J3.5 (Pin_5)
- net m8 Us: now reaches J4.1 (Pin_1)
- net m8 Us: now also D1.1 (K)
- net m8 GNDs: now reaches J4.3 (Pin_3)
- net m8 GNDs: now also D3.1 (K)
- new net Vcc+: C1.2, J3.1 (Pin_1), R14.2, U1.8 (Vs+), U2.3 (V+)
- new net Vcc-: C2.2, J3.3 (Pin_3), R15.1, U1.5 (Vs-), U2.4 (V-)
- new net m8 GNDp: D4.1 (K), J4.4 (Pin_4)
- new net m8 Up: D2.1 (K), J4.2 (Pin_2)
- new net rakout+: D1.2 (A), D2.2 (A), PS1.5 (+Vout), R12.2
- new net rakout-: D3.2 (A), D4.2 (A), D5.1 (K), PS1.4 (-Vout), R13.2
- no-connect marks 2 -> 3
Other:
- note added: "4.2V"
- note added: "Vcc+/2 at ref datasheet:8.3.7"
- note added: "housing GND?"
- note added: "m8 Up+- & m12 Up+- are connected in beckhoff"
- note removed: "Up is for Ext Sensor on analog input 1,2 we need Us to get to the beckhoff for processor logic field bus & analog i/0"
- note removed: "pwrout+/2 divider at ref datasheet:8.3.7"
- moved on the sheet: J4, J5, J6, J7

Commit message: end of day
Parts:
- removed U2: ${SIM.PARAMS}, symbol Simulation_SPICE:OPAMP
- added C3, C4: 104, 0603, symbol Device:C
- added U3: LM1458mx, Package_SO:SOIC-8_3.9x4.9mm_P1.27mm, symbol Device:Opamp_Dual
Connections:
- net GND: now also C3.1, C4.1, U3.1, U3.2 (-)
- net Vcc+: now also C2.2, U3.8 (V+)
- net Vcc-: now also C3.2, C4.2, U3.4 (V-); no longer C2.2
- net at R14.1, R15.2: now also U3.3 (+)
Other:
- note added: "for 7/15/26: m8, m12 connectors & footprints switch footprint ina825 footprint base pcbnew layout determine approx case dimensions based on footprints/connectors"
- note added: "housing GND? would be m8 shield as per beckhoff manual case will likely be Polycarbonate"
- note removed: "housing GND?"
- note removed: "tie pwrout- to devicecommon gnd? check m12 acode pinout -nope-"
- note removed: "with the ref divider sigout- and pwrout- are at two different potentials sigout- is directly between pwr +/-, it is gnd double check the beckoff manual"
- moved on the sheet: C1, C2, J3, R14, R15
