File: kicad/scribble.kicad_sch (KiCad schematic)
At the start: 14 parts

Commit message: Reorganized file structure
Parts:
- added SW1: SW_Push, symbol Switch:SW_Push
Connections:
- net at a5.: now also a6.
- net at a6.: no longer a5.
- net at a9.: now also a7.; no longer a2.
- net at a8.: now also a10.
- new net: a2., a9.
Changed lines of the file:
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@@
+	)
+	(rectangle
+		(start 151.765 100.965)
+		(end 168.275 132.08)
+		(stroke
+			(width 0)
+			(type default)
+		)
+		(fill
+			(type none)
+		)
 	)
 	(rectangle
@@
 		(fill
 			(type none)
+		)
+	)
+	(text "catpaw"
+		(exclude_from_sim no)
+		(at 155.194 99.314 0)
+		(effects
+			(font
+				(size 1.27 1.27)
+			)
 		)
 	)
@@
 		)
 		(instances
+			(project "scribble"
+				(path "/656593ca-6a57-45c5-a863-ae60861bb83b"
+					(reference "a?")
+					(unit 1)
+				)
+			)
 			(project "catpaw"
 				(path "/c6afa226-7a71-49a1-9fd2-6abf112b3631/10e6bb49-f350-49cb-8550-57ea3a57f8d7"
@@
 		)
 		(instances
+			(project "scribble"
+				(path "/656593ca-6a57-45c5-a863-ae60861bb83b"
+					(reference "a?")
+					(unit 1)
+				)
+			)
 			(project "catpaw"
 				(path "/c6afa226-7a71-49a1-9fd2-6abf112b3631/10e6bb49-f350-49cb-8550-57ea3a57f8d7"
@@
 		)
 		(instances
+			(project "scribble"
+				(path "/656593ca-6a57-45c5-a863-ae60861bb83b"
+					(reference "a?")
+					(unit 1)
+				)
+			)
 			(project "catpaw"
 				(path "/c6afa226-7a71-49a1-9fd2-6abf112b3631/10e6bb49-f350-49cb-8550-57ea3a57f8d7"
@@
 		)
 		(instances
+			(project "scribble"
+				(path "/656593ca-6a57-45c5-a863-ae60861bb83b"
+					(reference "a?")
+					(unit 1)
+				)
+			)
 			(project "catpaw"
 				(path "/c6afa226-7a71-49a1-9fd2-6abf112b3631/10e6bb49-f350-49cb-8550-57ea3a57f8d7"
@@
 		)
 		(instances
+			(project "scribble"
+				(path "/656593ca-6a57-45c5-a863-ae60861bb83b"
+					(reference "a?")
+					(unit 1)
+				)
+			)
 			(project "catpaw"
 				(path "/c6afa226-7a71-49a1-9fd2-6abf112b3631/10e6bb49-f350-49cb-8550-57ea3a57f8d7"
@@
 		)
 		(instances
+			(project "scribble"
+				(path "/656593ca-6a57-45c5-a863-ae60861bb83b"
+					(reference "a?")
+					(unit 1)
+				)
+			)
 			(project "catpaw"
 				(path "/c6afa226-7a71-49a1-9fd2-6abf112b3631/10e6bb49-f350-49cb-8550-57ea3a57f8d7"
@@
 		)
 		(instances
+			(project "scribble"
+				(path "/656593ca-6a57-45c5-a863-ae60861bb83b"
+					(reference "a?")
+					(unit 1)
+				)
+			)
 			(project "catpaw"
 				(path "/c6afa226-7a71-49a1-9fd2-6abf112b3631/10e6bb49-f350-49cb-8550-57ea3a57f8d7"
@@
 		)
 		(instances
+			(project "scribble"
+				(path "/656593ca-6a57-45c5-a863-ae60861bb83b"
+					(reference "a?")
+					(unit 1)
+				)
+			)
 			(project "catpaw"
 				(path "/c6afa226-7a71-49a1-9fd2-6abf112b3631/10e6bb49-f350-49cb-8550-57ea3a57f8d7"
@@
 		)
 		(instances
+			(project "scribble"
+				(path "/656593ca-6a57-45c5-a863-ae60861bb83b"
+					(reference "a?")
+					(unit 1)
+				)
+			)
 			(project "catpaw"
 				(path "/c6afa226-7a71-49a1-9fd2-6abf112b3631/10e6bb49-f350-49cb-8550-57ea3a57f8d7"
@@
 		)
 		(instances
+			(project "scribble"
+				(path "/656593ca-6a57-45c5-a863-ae60861bb83b"
+					(reference "a?")
+					(unit 1)
+				)
+			)
 			(project "catpaw"
 				(path "/c6afa226-7a71-49a1-9fd2-6abf112b3631/10e6bb49-f350-49cb-8550-57ea3a57f8d7"
@@
 		)
 		(instances
+			(project "scribble"
+				(path "/656593ca-6a57-45c5-a863-ae60861bb83b"
+					(reference "a?")
+					(unit 1)
+				)
+			)
 			(project "catpaw"
 				(path "/c6afa226-7a71-49a1-9fd2-6abf112b3631/10e6bb49-f350-49cb-8550-57ea3a57f8d7"
@@
 		)
 		(instances
+			(project "scribble"
+				(path "/656593ca-6a57-45c5-a863-ae60861bb83b"
+					(reference "a?")
+					(unit 1)
+				)
+			)
 			(project "catpaw"
 				(path "/c6afa226-7a71-49a1-9fd2-6abf112b3631/10e6bb49-f350-49cb-8550-57ea3a57f8d7"
 					(reference "a10")
+					(unit 1)
+				)
+			)
+		)
+	)
+	(symbol
+		(lib_id "Switch:SW_Push")
+		(at 92.71 55.88 90)
+		(unit 1)
+		(exclude_from_sim no)
+		(in_bom yes)
+		(on_board yes)
+		(dnp no)
+		(fields_autoplaced yes)
+		(property "Reference" "SW?"
+			(at 93.98 54.6099 90)
+			(effects
+				(font
+					(size 1.27 1.27)
+				)
+				(justify right)
+			)
+		)
+		(property "Value" "SW_Push"
+			(at 93.98 57.1499 90)
+			(effects
+				(font
+					(size 1.27 1.27)
+				)
+				(justify right)
+			)
+		)
+		(property "Footprint" ""
+			(at 87.63 55.88 0)
+			(effects
+				(font
+					(size 1.27 1.27)
+				)
+				(hide yes)
+			)
+		)
+		(property "Datasheet" "~"
+			(at 87.63 55.88 0)
+			(effects
+				(font
+					(size 1.27 1.27)
+				)
+				(hide yes)
+			)
+		)
+		(property "Description" "Push button switch, generic, two pins"
+			(at 92.71 55.88 0)
+			(effects
+				(font
+					(size 1.27 1.27)
+				)
+				(hide yes)
+			)
+		)
+		(pin "2"
+		)
+		(pin "1"
+		)
+		(instances
+			(project ""
+				(path "/656593ca-6a57-45c5-a863-ae60861bb83b"
+					(reference "SW1")
+					(unit 1)
+				)
+			)
+			(project "catpaw"
+				(path "/c6afa226-7a71-49a1-9fd2-6abf112b3631/10e6bb49-f350-49cb-8550-57ea3a57f8d7"
+					(reference "SW?")
 					(unit 1)
 				)
@@
 		)
 		(instances
+			(project "scribble"
+				(path "/656593ca-6a57-45c5-a863-ae60861bb83b"
+					(reference "a?")
+					(unit 1)
+				)
+			)
 			(project "catpaw"
 				(path "/c6afa226-7a71-49a1-9fd2-6abf112b3631/10e6bb49-f350-49cb-8550-57ea3a57f8d7"
@@
 		)
 		(instances
+			(project "scribble"
+				(path "/656593ca-6a57-45c5-a863-ae60861bb83b"
+					(reference "a?")
+					(unit 1)
+				)
+			)
 			(project "catpaw"
 				(path "/c6afa226-7a71-49a1-9fd2-6abf112b3631/10e6bb49-f350-49cb-8550-57ea3a57f8d7"
@@
 		)
 	)
+	(sheet_instances
+		(path "/"
+			(page "1")
+		)
+	)
+	(embedded_fonts no)
 )

Commit message: Footprints assigned
Parts:
- renumbered SW1 to SW2
Connections:
- net at a5.: now also a6.
- net at a6.: no longer a5.
- net at a9.: now also a7.; no longer a2.
- net at a8.: now also a10.
- new net: a2., a9.
Changed lines of the file:
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@@
 		(dnp no)
 		(fields_autoplaced yes)
-		(property "Reference" "SW?"
+		(property "Reference" "SW2"
 			(at 93.98 54.6099 90)
 			(effects
@@
 			(project "catpaw"
 				(path "/c6afa226-7a71-49a1-9fd2-6abf112b3631/10e6bb49-f350-49cb-8550-57ea3a57f8d7"
-					(reference "SW?")
+					(reference "SW2")
 					(unit 1)
 				)
