File: kicad/catpaw.kicad_pcb (KiCad board)
At the start: 2 copper layers, 79 x 75 mm, 37 parts, among them J1 Conn_01x01_Socket_red, J2 Conn_01x01_Socket_black, J3 m12,Acode,5pin,femalesocket (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, J4 m8, 4Pin Supply Connector FEM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, SW1 1MD1T1B1M6QES, U1 INA826, U2 LM1458mx

Commit message: added rev01 buildout photos
Parts:
- moved J3 4.51 mm to (179.0, 93.6)
Routing:
- net /In+ Analog Input: track 11.5 -> 16.1 mm, vias 0 -> 1
- net /Vcc-: track 55.9 -> 60.3 mm
- net /Vcc+: track 60.6 -> 56.5 mm
- removed copper zone on F.Cu, net /Vcc+
Other:
- board text added: "amphenol gives 2mm to pcb edge see m12 tech datasheet choosing 4.00mm setback"
- board text removed: "amphenol gives 5.8mm to pcb edge see m12 tech datasheet"
Changed lines of the file:
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@@
 	(footprint "kyuditsky_kicad:M12A05PFFRSF7003"
 		(layer "F.Cu")
-		(at 174.444 93.556 90)
+		(at 178.954 93.602 90)
 		(descr "M12A-05PFFR-SF7003")
 		(tags "Connector")
@@
 	)
 	(gr_line
+		(start 188.722 102.87)
+		(end 184.722 102.87)
+		(stroke
+			(width 0.05)
+			(type solid)
+		)
+		(layer "User.2")
+	)
+	(gr_line
 		(start 188.712 78.324)
 		(end 188.712 95.324)
@@
 		)
 	)
-	(gr_text "amphenol gives 5.8mm to pcb edge\nsee m12 tech datasheet"
+	(gr_text "amphenol gives 2mm to pcb edge\nsee m12 tech datasheet\nchoosing 4.00mm setback"
 		(at 191.008 113.03 0)
 		(layer "User.2")
@@
 	)
 	(segment
+		(start 167.132 84.436372)
+		(end 163.966314 81.270686)
+		(width 0.75)
+		(layer "F.Cu")
+		(net 1)
+	)
+	(segment
 		(start 154.94 73.66)
 		(end 152.4 71.12)
@@
 	)
 	(segment
-		(start 168.148 77.581)
-		(end 169.148 77.581)
+		(start 167.132 92.583)
+		(end 167.132 84.436372)
 		(width 0.75)
 		(layer "F.Cu")
@@
 	)
 	(segment
-		(start 167.132 84.436372)
-		(end 163.966314 81.270686)
+		(start 168.148 77.581)
+		(end 169.148 77.581)
 		(width 0.75)
 		(layer "F.Cu")
@@
 	)
 	(segment
-		(start 168.105 93.556)
-		(end 167.132 92.583)
-		(width 0.75)
-		(layer "F.Cu")
-		(net 1)
-	)
-	(segment
 		(start 167.656 77.581)
 		(end 168.148 77.581)
@@
 	)
 	(segment
-		(start 174.444 93.556)
-		(end 169.291 93.556)
+		(start 155.579 73.66)
+		(end 155.448 73.66)
 		(width 0.75)
 		(layer "F.Cu")
@@
 	)
 	(segment
-		(start 155.579 73.66)
-		(end 155.448 73.66)
+		(start 156.355628 73.66)
+		(end 155.579 73.66)
 		(width 0.75)
 		(layer "F.Cu")
@@
 	)
 	(segment
-		(start 167.132 92.583)
-		(end 167.132 84.436372)
+		(start 168.151 93.602)
+		(end 169.245 93.602)
 		(width 0.75)
 		(layer "F.Cu")
@@
 	)
 	(segment
-		(start 156.355628 73.66)
-		(end 155.579 73.66)
+		(start 169.148 77.581)
+		(end 169.672 78.105)
 		(width 0.75)
 		(layer "F.Cu")
@@
 	)
 	(segment
-		(start 169.291 93.556)
-		(end 168.105 93.556)
+		(start 169.291 93.599)
+		(end 170.307 93.599)
 		(width 0.75)
 		(layer "F.Cu")
@@
 	)
 	(segment
-		(start 169.148 77.581)
-		(end 169.672 78.105)
+		(start 142.24 71.12)
+		(end 152.4 71.12)
 		(width 0.75)
 		(layer "F.Cu")
@@
 	)
 	(segment
-		(start 142.24 71.12)
-		(end 152.4 71.12)
+		(start 168.151 93.602)
+		(end 167.132 92.583)
 		(width 0.75)
 		(layer "F.Cu")
@@
 	)
 	(via
-		(at 169.291 93.556)
+		(at 168.529 93.599)
 		(size 0.6)
 		(drill 0.3)
@@
 	)
 	(via
-		(at 170.688 94.996)
+		(at 142.24 71.12)
 		(size 0.6)
 		(drill 0.3)
@@
 	)
 	(via
-		(at 142.24 71.12)
+		(at 169.418 93.599)
 		(size 0.6)
 		(drill 0.3)
@@
 	)
 	(via
-		(at 170.688 95.758)
+		(at 170.307 93.599)
 		(size 0.6)
 		(drill 0.3)
@@
 	)
 	(via
-		(at 180.213 92.075)
+		(at 177.927 90.551)
 		(size 0.6)
 		(drill 0.3)
@@
 	)
 	(via
-		(at 180.213 93.599)
+		(at 179.451 90.551)
 		(size 0.6)
 		(drill 0.3)
@@
 	)
 	(via
-		(at 177.165 91.059)
+		(at 184.912 93.853)
 		(size 0.6)
 		(drill 0.3)
@@
 	)
 	(via
-		(at 178.689 91.059)
+		(at 184.912 92.329)
 		(size 0.6)
 		(drill 0.3)
@@
 	)
 	(via
-		(at 177.927 91.059)
+		(at 184.912 93.091)
 		(size 0.6)
 		(drill 0.3)
@@
 	)
 	(via
-		(at 180.213 92.837)
+		(at 178.689 90.551)
 		(size 0.6)
 		(drill 0.3)
@@
 	)
 	(segment
-		(start 176.657 78.105)
-		(end 175.26 78.105)
+		(start 150.245 78.74)
+		(end 160.02 78.74)
 		(width 0.75)
 		(layer "F.Cu")
@@
 	)
 	(segment
-		(start 160.02 78.74)
-		(end 166.116 84.836)
+		(start 176.657 78.105)
+		(end 175.26 78.105)
 		(width 0.75)
 		(layer "F.Cu")
@@
 	)
 	(segment
-		(start 175.635 99.187)
-		(end 177.98 96.842)
-		(width 0.75)
-		(layer "F.Cu")
-		(net 3)
-	)
-	(segment
 		(start 170.434 99.187)
-		(end 175.635 99.187)
+		(end 180.441 99.187)
 		(width 0.75)
 		(layer "F.Cu")
@@
 	)
 	(segment
-		(start 166.116 84.836)
-		(end 166.116 94.869)
+		(start 160.02 78.74)
+		(end 166.116 84.836)
 		(width 0.75)
 		(layer "F.Cu")
@@
 	)
 	(segment
-		(start 150.245 78.74)
-		(end 160.02 78.74)
+		(start 175.26 78.105)
+		(end 168.656 84.709)
 		(width 0.75)
 		(layer "F.Cu")
@@
 	)
 	(segment
-		(start 175.26 78.105)
-		(end 168.656 84.709)
+		(start 166.116 84.836)
+		(end 166.116 94.869)
+		(width 0.75)
+		(layer "F.Cu")
+		(net 3)
+	)
+	(segment
+		(start 180.441 99.187)
+		(end 182.49 97.138)
 		(width 0.75)
 		(layer "F.Cu")
@@
 	)
 	(segment
-		(start 174.444 96.842)
+		(start 171.704 91.186)
 		(end 171.704 94.102)
 		(width 0.75)
-		(layer "B.Cu")
+		(layer "F.Cu")
 		(net 14)
 	)
 	(segment
-		(start 172.974 89.916)
-		(end 172.974 89.646)
+		(start 171.704 94.102)
+		(end 174.74 97.138)
 		(width 0.75)
-		(layer "B.Cu")
+		(layer "F.Cu")
 		(net 14)
 	)
 	(segment
-		(start 171.704 91.186)
-		(end 172.974 89.916)
+		(start 174.74 97.138)
+		(end 178.954 97.138)
+		(width 0.75)
+		(layer "F.Cu")
+		(net 14)
+	)
+	(via
+		(at 171.704 91.186)
+		(size 0.6)
+		(drill 0.3)
+		(layers "F.Cu" "B.Cu")
+		(net 14)
+	)
+	(segment
+		(start 172.974 89.916)
+		(end 172.974 89.646)
 		(width 0.75)
 		(layer "B.Cu")
@@
 	)
 	(segment
-		(start 171.704 94.102)
-		(end 171.704 91.186)
+		(start 171.704 91.186)
+		(end 172.974 89.916)
 		(width 0.75)
 		(layer "B.Cu")
@@
 	)
 	(zone
-		(net 1)
-		(net_name "/Vcc+")
+		(net 2)
+		(net_name "GND")
 		(layers "F.Cu" "B.Cu")
 		(hatch edge 0.5)
-		(priority 4)
-		(connect_pads yes
+		(connect_pads
 			(clearance 0.5)
 		)
@@
 			(thermal_bridge_width 0.5)
 			(smoothing fillet)
-			(radius 0.65)
+			(radius 2)
 		)
 		(polygon
 			(pts
-				(xy 167.894 91.948) (xy 175.387 91.948) (xy 175.387 94.234) (xy 172.212 95.504) (xy 170.561 96.774)
-				(xy 167.894 94.488)
+				(xy 187.706 43.942) (xy 187.706 112.776) (xy 162.306 112.776) (xy 162.217212 88.653771) (xy 160.137579 85.375582)
+				(xy 155.477395 83.159769) (xy 152.203998 82.433994) (xy 136.652 82.55) (xy 136.652 65.744422) (xy 135.5725 63.246)
+				(xy 132.334 60.198) (xy 132.334 57.3405) (xy 131.537477 55.86569) (xy 129.229744 54.352422) (xy 127.540621 53.848)
+				(xy 110.998 53.975) (xy 110.998 44.069)
 			)
 		)
 	)
 	(zone
-		(net 2)
-		(net_name "GND")
-		(layers "F.Cu" "B.Cu")
+		(net 1)
+		(net_name "/Vcc+")
+		(layer "B.Cu")
 		(hatch edge 0.5)
-		(connect_pads
+		(priority 4)
+		(connect_pads yes
 			(clearance 0.5)
 		)
@@
 			(thermal_bridge_width 0.5)
 			(smoothing fillet)
-			(radius 2)
+			(radius 0.65)
 		)
 		(polygon
 			(pts
-				(xy 187.706 43.942) (xy 187.706 112.776) (xy 162.306 112.776) (xy 162.217212 88.653771) (xy 160.137579 85.375582)
-				(xy 155.477395 83.159769) (xy 152.203998 82.433994) (xy 136.652 82.55) (xy 136.652 65.744422) (xy 135.5725 63.246)
-				(xy 132.334 60.198) (xy 132.334 57.3405) (xy 131.537477 55.86569) (xy 129.229744 54.352422) (xy 127.540621 53.848)
-				(xy 110.998 53.975) (xy 110.998 44.069)
+				(xy 167.89321 91.8953) (xy 179.83121 92.0223) (xy 179.83121 94.3083) (xy 172.212 96.012) (xy 169.545 96.012)
+				(xy 167.89321 94.4353)
 			)
 		)

Commit message: added vac scope images
Other:
- board text added: "LED needs reworked. will only light if both PSU is powered AND catpaw internals are powered it is not always the most intuitive haptic"
Changed lines of the file:
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@@
+		)
+	)
+	(gr_text "LED needs reworked.\nwill only light if both PSU is powered AND catpaw internals are powered\nit is not always the most intuitive haptic"
+		(at 97.282 28.829 0)
+		(layer "User.2")
+		(effects
+			(font
+				(size 1.5 1.5)
+				(thickness 0.3)
+				(bold yes)
+			)
+			(justify left bottom)
 		)
 	)

Commit message: Begin Rev1.1
Other:
- board text added: "09/16/26"
- board text added: "rev1.1"
- board text removed: "07/20/26"
Changed lines of the file:
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@@
 		)
 	)
-	(gr_text "07/20/26"
+	(gr_text "09/16/26"
 		(at 207.01 193.802 0)
 		(layer "User.2")
@@
 				(bold yes)
 			)
+			(justify left bottom)
+		)
+	)
+	(gr_text "rev1.1"
+		(at 187.706 190.373 0)
+		(layer "User.2")
+		(effects
+			(font
+				(size 1.5 1.5)
+				(thickness 0.3)
+				(bold yes)
+			)

Commit message: added new bode plots
Parts:
- moved F1 14.0 mm to (153.3, 110.2)
- moved J3 0.50 mm to (178.5, 93.6)
Routing:
- net Net-(F1-Pad1): track 13.6 -> 27.6 mm
- net Net-(PS1-AC(L)): track 17.1 -> 7.55 mm
Other:
- board text added: "catpaw rev1.1 sep26 //keyudits"
- board text removed: "amphenol gives 2mm to pcb edge see m12 tech datasheet choosing 4.00mm setback"
- board text removed: "catpaw rev01 jul26 //keyudits"
- board text removed: "move f1 away from exposed vac pad (8mm)"
Changed lines of the file:
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@@
 	(footprint "kyuditsky_kicad:FUSC10131X312N"
 		(layer "F.Cu")
-		(at 139.319 110.236)
+		(at 153.289 110.236)
 		(descr "0461002")
 		(tags "Fuse")
@@
 	(footprint "kyuditsky_kicad:M12A05PFFRSF7003"
 		(layer "F.Cu")
-		(at 178.954 93.602 90)
+		(at 178.454 93.602 90)
 		(descr "M12A-05PFFR-SF7003")
 		(tags "Connector")
@@
 	)
 	(gr_line
-		(start 188.712 95.324)
-		(end 176.212 95.324)
-		(stroke
-			(width 0.1)
-			(type solid)
-		)
-		(layer "User.2")
-	)
-	(gr_line
 		(start 188.712 78.324)
 		(end 188.712 61.324)
@@
 	(gr_line
 		(start 188.722 102.87)
-		(end 184.722 102.87)
+		(end 184.222 102.87)
 		(stroke
 			(width 0.05)
@@
 		(layer "User.2")
 	)
-	(gr_text "catpaw rev01 jul26\n//keyudits"
+	(gr_text "catpaw rev1.1 sep26\n//keyudits"
 		(at 185.42 110.49 0)
 		(layer "F.SilkS")
@@
 		)
 	)
-	(gr_text "amphenol gives 2mm to pcb edge\nsee m12 tech datasheet\nchoosing 4.00mm setback"
-		(at 191.008 113.03 0)
-		(layer "User.2")
-		(effects
-			(font
-				(size 1 1)
-				(thickness 0.25)
-				(bold yes)
-			)
-			(justify left bottom)
-		)
-	)
 	(gr_text "rac20-24sk/277"
 		(at 160.274 70.993 90)
@@
 		)
 	)
-	(gr_text "move f1 away from exposed vac pad (8mm)"
-		(at 130.302 117.983 0)
-		(layer "User.2")
-		(effects
-			(font
-				(size 1 1)
-				(thickness 0.25)
-				(bold yes)
-			)
-			(justify left bottom)
-		)
-	)
 	(gr_text "rev1.1"
 		(at 187.706 190.373 0)
@@
 	)
 	(segment
-		(start 150.362 110.236)
-		(end 157.7265 102.8715)
+		(start 157.7265 109.7925)
+		(end 157.283 110.236)
 		(width 1.5)
 		(layer "F.Cu")
@@
 	)
 	(segment
-		(start 143.694 110.236)
-		(end 150.362 110.236)
+		(start 157.7265 102.8715)
+		(end 157.7265 109.7925)
 		(width 1.5)
 		(layer "F.Cu")
@@
 	(segment
 		(start 125.222 107.95)
-		(end 125.222 105.019)
+		(end 127.508 110.236)
 		(width 1.5)
 		(layer "F.Cu")
@@
 	)
 	(segment
-		(start 134.944 110.236)
-		(end 127.508 110.236)
+		(start 125.222 105.019)
+		(end 125.222 107.95)
 		(width 1.5)
 		(layer "F.Cu")
@@
 	(segment
 		(start 127.508 110.236)
-		(end 125.222 107.95)
+		(end 148.914 110.236)
 		(width 1.5)
 		(layer "F.Cu")
@@
 		(min_thickness 0.25)
 		(filled_areas_thickness no)
-		(fill yes
+		(fill
 			(thermal_gap 0.5)
 			(thermal_bridge_width 0.5)
@@
 		(min_thickness 0.25)
 		(filled_areas_thickness no)
-		(fill yes
+		(fill
 			(thermal_gap 0.5)
 			(thermal_bridge_width 0.5)
@@
 		(min_thickness 0.25)
 		(filled_areas_thickness no)
-		(fill yes
+		(fill
 			(thermal_gap 0.5)
 			(thermal_bridge_width 0.5)
@@
 		(min_thickness 0.25)
 		(filled_areas_thickness no)
-		(fill yes
+		(fill
 			(thermal_gap 0.5)
 			(thermal_bridge_width 0.5)
@@
 		(min_thickness 0.25)
 		(filled_areas_thickness no)
-		(fill yes
+		(fill
 			(thermal_gap 0.5)
 			(thermal_bridge_width 0.5)

Commit message: rev1.1 updates
Parts:
- added R8: 30.1k, Resistor_SMD:R_0805_2012Metric_Pad1.20x1.40mm_HandSolder, B.Cu at (156.2, 94.5)
- R13: value 1k -> 2.2k
- R7: value 60.4k -> 30.1k
- VCC: renamed from R18; footprint Resistor_THT:R_Axial_DIN0204_L3.6mm_D1.6mm_P2.54mm_Vertical -> TestPoint:TestPoint_2Pads_Pitch2.54mm_Drill0.8mm
- VEE: renamed from R19; footprint Resistor_THT:R_Axial_DIN0204_L3.6mm_D1.6mm_P2.54mm_Vertical -> TestPoint:TestPoint_2Pads_Pitch2.54mm_Drill0.8mm
- moved R13 8.26 mm to (139.6, 63.0), turned to -90 degrees
- moved R7 6.55 mm to (156.2, 86.4)
- moved R10 3.18 mm to (159.4, 93.6)
- moved R9 3.18 mm to (159.4, 87.5)
- moved R21 1.72 mm to (173.7, 90.2)
- moved R1 0.89 mm to (138.9, 86.5)
- moved R2 0.89 mm to (144.9, 86.5)
- moved R3 0.89 mm to (150.8, 86.5)
- moved R4 0.89 mm to (139.0, 95.1)
- moved R5 0.89 mm to (144.9, 95.1)
- moved R6 0.89 mm to (150.8, 95.1)
- moved C4 0.57 mm to (146.9, 78.9)
- renumbered R9 to R10, R10 to R11, VCC to R17, VEE to R20, R11 to R21, R8 to R9
Connections:
- R10 pad 1: Net-(R6-Pad1) -> Net-(R10-Pad1)
- R13 pad 2: /m8 GNDp -> GND
- R6 pad 1: Net-(R6-Pad1) -> Net-(R10-Pad1)
- R7 pad 1: Net-(R3-Pad1) -> GND
- R7 pad 2: Net-(R6-Pad1) -> Net-(R3-Pad1)
Routing:
- net Net-(U2B-+): track 28.3 -> 21.3 mm
- net Net-(R10-Pad1): track 0.00 -> 6.71 mm
- net Net-(R6-Pad1): track 6.14 -> 0.00 mm
- net /VACin+: track 50.3 -> 47.2 mm
- net Net-(U1--): track 7.24 -> 4.24 mm
- net Net-(U1-+): track 7.24 -> 4.24 mm
- net /m8 GNDp: track 55.2 -> 52.4 mm
- net /In+ Analog Input: track 16.1 -> 13.5 mm
- net /Vcc-: track 60.3 -> 58.0 mm, vias 6 -> 0
- net /Vcc+: track 56.5 -> 55.8 mm, vias 8 -> 4
- net Net-(D5-A): track 54.9 -> 54.3 mm
- net GND: vias 135 -> 150
Other:
- board text added: "jump for testing only"
- board text removed: "LED needs reworked. will only light if both PSU is powered AND catpaw internals are powered it is not always the most intuitive haptic"
- board text removed: "adjust vcc/vee jumper footprint to 2.54 vertical header pins"
- board text removed: "rac15-24sk/480"
