File: kicad/sim/sim.kicad_sch (KiCad schematic)
At the start: 14 parts, among them U1 INA826

Commit message: updated sim.kicad
Parts:
- added V3: dc=12, symbol Simulation_SPICE:VDC
- V2: value 24 -> dc=12
Connections:
- net 0: now also V2.2, V3.1
- net Vcc-: now also V3.2; no longer V2.2
- net VACin+ renamed input
- net sigout+ renamed output
Other:
- note added: ".ac dec 10 1 10000k"
- note removed: ".ac dec 10 1 100000k"
- moved on the sheet: V2
