File: kicad/Rev1-1-fatpaw/sim/sim.kicad_sch (KiCad schematic)
At the start: 15 parts, among them U1 INA826

Commit message: forked catpaw-rev2, updated ina826 spice model
Other:
- note added: ".ac dec 10 1 1000k"
- note removed: ".ac dec 10 1 10000k"
Changed lines of the file:
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@@
 	(generator_version "9.0")
 	(paper "A4")
-	(text ".ac dec 10 1 10000k"
+	(text ".ac dec 10 1 1000k"
 		(exclude_from_sim no)
 		(at 54.864 113.538 0)
@@
 			)
 		)
-		(property "Sim.Library" "INA826_sbomc48/ina826.lib"
+		(property "Sim.Library" "INA826_sbomc48/ina826_updated.lib"
 			(at 166.37 96.52 0)
 			(effects
@@
 			)
 		)
-		(property "Sim.Pins" "1=IN- 2=RG+ 3=RG- 4=IN+ 5=GND 6=REF 7=OUT 8=VDD"
+		(property "Sim.Pins" "1=IN- 2=RG+ 3=RG- 4=IN+ 5=VNEGP 6=REF 7=OUT 8=VDD"
 			(at 166.37 96.52 0)
 			(effects
