File: kicad/Rev2-0-catpaw/catpaw2.kicad_sch (KiCad schematic)
At the start: 33 parts, among them J1 Conn_01x01_Socket_red, J2 Conn_01x01_Socket_black, J3 m12,Acode,5pin,femalesocket (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, J4 Conn_01x03_Pin, J5 m8, 4Pin Supply Connector Bec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, J6 m12,Acode,5pin,femalesocket B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, J7 m12,Acode,5pin,femalesocket C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, U1 INA826, U2 LM1458mx

Commit message: routed rev2.0
Parts:
- D5: footprint LED_THT:LED_D5.0mm_Horizontal_O1.27mm_Z3.0mm -> LED_THT:LED_D3.0mm_Horizontal_O1.27mm_Z2.0mm
- J4: footprint (none) -> Connector_PinHeader_2.54mm:PinHeader_1x03_P2.54mm_Vertical
Changed lines of the file:
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@@
 			)
 		)
-		(property "Footprint" "LED_THT:LED_D5.0mm_Horizontal_O1.27mm_Z3.0mm"
+		(property "Footprint" "LED_THT:LED_D3.0mm_Horizontal_O1.27mm_Z2.0mm"
 			(at 256.54 110.49 0)
 			(effects
@@
 			)
 		)
-		(property "Footprint" ""
+		(property "Footprint" "Connector_PinHeader_2.54mm:PinHeader_1x03_P2.54mm_Vertical"
 			(at 151.13 87.63 0)
 			(effects

Commit message: built catpaw rev2.0
Other:
- note added: "09/21/26"
- note added: "10/14/26 bench measurements match"
- note removed: "09/16/26"
- note removed: "update: 07/20/26"
- moved on the sheet: J1, J2, J3, J4, R1, R10, R11, R2, R21, R3, R4, R5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
